File: PCB/PS-microCard PCB.kicad_sch (KiCad schematic)
At the start: 0 parts

Commit message: Stage 7: First prototype pcb board
Parts:
- added C1, C13, C25, C26, C4, C6: 4.7u, Capacitor_SMD:C_0402_1005Metric, symbol Device:C
- added C10, C11, C12, C14, C15, C16, C17, C18, C20, C21, C22, C5, C7, C8, C9: 100n, Capacitor_SMD:C_0402_1005Metric, symbol Device:C
- added C19: 10u, Capacitor_SMD:C_0805_2012Metric, symbol Device:C
- added C2, C3: 15p, Capacitor_SMD:C_0402_1005Metric, symbol Device:C
- added C23, C27: 1u, Capacitor_SMD:C_0402_1005Metric, symbol Device:C
- added C24: 4.7u, Capacitor_SMD:C_0805_2012Metric, symbol Device:C
- added J1: Oled Socket, Connector_PinSocket_2.54mm:PinSocket_1x06_P2.54mm_Vertical, symbol Connector_Generic:Conn_01x06
- added J3: MEM2052-00-195-00-A_REVA, footprints:GCT_MEM2052-00-195-00-A_REVA, symbol MEM2052-00-195-00-A_REVA:MEM2052-00-195-00-A_REVA
- added J4: 10118194-0001LF, footprints:AMPHENOL_10118194-0001LF, symbol 10118194-0001LF:10118194-0001LF
- added J6: JST Debug Connector, Connector_JST:JST_SH_SM03B-SRSS-TB_1x03-1MP_P1.00mm_Horizontal, symbol Connector_Generic_MountingPin:Conn_01x03_MountingPin
- added L1: 3.3u, footprints:L_pol_2016, symbol Device:L
- added R1, R3: DNF, Resistor_SMD:R_0402_1005Metric, symbol Device:R
- added R10, R8: 10k, Resistor_SMD:R_0402_1005Metric, symbol Device:R
- added R11: 1K, Resistor_SMD:R_0402_1005Metric, symbol Device:R
- added R12, R13, R14, R15, R16: 47, Resistor_SMD:R_0402_1005Metric, symbol Device:R
- added R17, R18, R19, R5, R9: 1k, Resistor_SMD:R_0402_1005Metric, symbol Device:R
- added R2: 0, Resistor_SMD:R_0402_1005Metric, symbol Device:R
- added R4: 33, Resistor_SMD:R_0402_1005Metric, symbol Device:R
- added R6, R7: 27, Resistor_SMD:R_0402_1005Metric, symbol Device:R
- added S1, S2: USLPT2819DT2TR, footprints:SW_USLPT2819DT2TR, symbol USLPT2819DT2TR:USLPT2819DT2TR
- added SW1, SW2: FSM4JSMA, footprints:TE_FSM4JSMA, symbol FSM4JSMA:FSM4JSMA
- added TP1: PS1_DATA, footprints:Pad_kontaktowy_PS1_dane, symbol Connector:TestPoint
- added TP2: PS1_CMD, footprints:Pad_kontaktowy_PS1_dane, symbol Connector:TestPoint
- added TP3: PS1_CS, footprints:Pad_kontaktowy_PS1_dane, symbol Connector:TestPoint
- added TP4: PS1_SCK, footprints:Pad_kontaktowy_PS1_dane, symbol Connector:TestPoint
- added TP5: PS1_ACK, footprints:Pad_kontaktowy_PS1_dane, symbol Connector:TestPoint
- added TP6: PS1_7V5, footprints:Pad_kontaktowy_PS1_zasilanie, symbol Connector:TestPoint
- added TP7: PS1_GND, footprints:Pad_kontaktowy_PS1_zasilanie, symbol Connector:TestPoint
- added TP8: PS1_3V5, footprints:Pad_kontaktowy_PS1_zasilanie, symbol Connector:TestPoint
- added U1: W25Q128JVS, Package_SO:SOIC-8_5.3x5.3mm_P1.27mm, symbol Memory_Flash:W25Q128JVS
- added U2: RP2350_60QFN, footprints:RP2350-QFN-60-1EP_7x7_P0.4mm_EP3.4x3.4mm_ThermalVias, symbol MCU_RaspberryPi_RP2350:RP2350_60QFN
- added U3: TPS2113APWR, footprints:TPS2113-SOP65P640X120-8N, symbol TPS2113APWR:TPS2113APWR
- added U4: TLV75533PDBVR, footprints:TLV75533PDBVR-SOT95P280X145-5N, symbol TLV75533PDBVR:TLV75533PDBVR
- added U5: TPS7A2033PDBVR, footprints:TPS7A2033PDBVR-SOT95P280X145-5N, symbol TPS7A2033PDBVR:TPS7A2033PDBVR
- added Y1: ABM8-272-T3, footprints:XTAL_ABM8-272-T3, symbol ABM8-272-T3:ABM8-272-T3
Connections:
- new net: R17.1, SW1.3, SW1.4
- new net: R11.2, S1.3, S1.4
- new net: C27.1, TP8.1, U5.1 (IN), U5.3 (EN)
- new net: R7.2, U2.51 (USB_DM)
- new net: R6.1, U2.52 (USB_DP)
- new net: R9.1, U3.4 (ILIM)
- new net: C3.2, R5.1, Y1.1
- new net: R18.1, SW2.3, SW2.4
- new net +1V1: C11.1, C13.1, C15.1, C4.1, L1.1, U2.23 (DVDD), U2.39 (DVDD), U2.50 (VREG_FB), U2.6 (DVDD)
- new net +3V3: C1.1, C10.1, C12.1, C14.1, C16.1, C17.1, C18.1, C19.1, C22.1, C24.1, C5.1, C7.1, C8.1, C9.1, J1.1 (Pin_1), J3.P4 (VDD), R10.1, R3.1, R4.2, R8.2, U1.8 (VCC), U2.1 (IOVDD), U2.11 (IOVDD), U2.20 (IOVDD), U2.30 (IOVDD), U2.38 (IOVDD), U2.44 (ADC_AVDD), U2.45 (IOVDD), U2.49 (VREG_VIN), U2.53 (USB_OTP_VDD), U2.54 (QSPI_IOVDD), U3.7 (OUT)
- new net FLASH_SS: R1.1, R2.1, R3.2, U1.1 (~{CS})
- new net GND: C1.2, C10.2, C11.2, C12.2, C13.2, C14.2, C15.2, C16.2, C17.2, C18.2, C19.2, C2.1, C20.1, C21.2, C22.2, C23.1, C24.2, C25.1, C26.2, C27.2, C3.1, C4.2, C5.2, C6.2, C7.2, C8.2, C9.2, J1.2 (Pin_2), J3.G1 (SHIELD_GND), J3.G2 (SHIELD_GND), J3.G3 (SHIELD_GND), J3.G4 (SHIELD_GND), J3.P6 (VSS), J4.5 (GND), J4.SH1 (SHIELD), J4.SH2 (SHIELD), J4.SH3 (SHIELD), J4.SH4 (SHIELD), J4.SH5 (SHIELD), J4.SH6 (SHIELD), J6.2 (Pin_2), J6.MP (MountPin), R11.1, R9.2, S2.1, S2.2, SW1.1, SW1.2, SW2.1, SW2.2, TP7.1, U1.4 (GND), U2.47 (VREG_PGND), U2.61 (GND), U3.2 (~{EN}), U3.5 (GND), U4.2 (GND), U5.2 (GND), Y1.2 (GND), Y1.4 (GND)
- new net GPIO0: R1.2, U2.2 (GPIO0)
- new net Left Button: R18.2, U2.12 (GPIO8)
- new net OLED_CS: J1.6 (Pin_6), U2.17 (GPIO13)
- new net OLED_D/C: J1.5 (Pin_5), U2.16 (GPIO12)
- new net OLED_MOSI: J1.4 (Pin_4), U2.15 (GPIO11)
- new net OLED_SCK: J1.3 (Pin_3), U2.14 (GPIO10)
- new net PS1_3V3: C20.2, C26.1, U3.3 (VSNS), U3.8 (IN1), U5.5 (OUT)
- new net PS1_ACK: R16.2, U2.4 (GPIO2)
- new net PS1_ACK_DBG: R16.1, TP5.1
- new net PS1_CMD: R13.1, U2.8 (GPIO5)
- new net PS1_CMD_DBG: R13.2, TP2.1
- new net PS1_CS: R14.1, U2.7 (GPIO4)
- new net PS1_CS_DBG: R14.2, TP3.1
- new net PS1_DATA: R12.2, U2.9 (GPIO6)
- new net PS1_DATA_DBG: R12.1, TP1.1
- new net PS1_SCK: R15.1, U2.5 (GPIO3)
- new net PS1_SCK_DBG: R15.2, TP4.1
- new net QSPI_SCLK: U1.6 (CLK), U2.56 (QSPI_SCLK)
- new net QSPI_SD0: U1.5 (DI/IO_{0}), U2.57 (QSPI_SD0)
- new net QSPI_SD1: U1.2 (DO/IO_{1}), U2.59 (QSPI_SD1)
- new net QSPI_SD2: U1.3 (~{WP}/IO_{2}), U2.58 (QSPI_SD2)
- new net QSPI_SD3: U1.7 (~{HOLD}/~{RESET}/IO_{3}), U2.55 (QSPI_SD3)
- new net QSPI_SS: R19.1, R2.2, U2.60 (QSPI_SS)
- new net RUN: S1.1, S1.2, U2.26 (RUN)
- new net Right Button: R17.2, U2.13 (GPIO9)
- new net SD_CS: J3.P2 (CD/DAT3), R8.1, U2.33 (GPIO21)
- new net SD_DETECT: J3.P9 (CD_PIN), R10.2, U2.36 (GPIO24)
- new net SD_MISO: J3.P7 (DAT0), U2.32 (GPIO20)
- new net SD_MOSI: J3.P3 (CMD), U2.35 (GPIO23)
- new net SD_SCK: J3.P5 (CLK), U2.34 (GPIO22)
- new net SWCLK: J6.1 (Pin_1), U2.24 (SWCLK)
- new net SWD: J6.3 (Pin_3), U2.25 (SWD)
- new net USB_3V3: C21.1, C25.2, U3.6 (IN2), U4.5 (OUT)
- new net USB_BOOT: R19.2, S2.3, S2.4
- new net USB_D+: J4.3 (D+), R6.2
- new net USB_D-: J4.2 (D-), R7.1
- new net VBUS: C23.2, J4.1 (VCC), U4.1 (IN), U4.3 (EN)
- new net VREG_AVDD: C6.1, R4.1, U2.46 (VREG_AVDD)
- new net VREG_LX: L1.2, U2.48 (VREG_LX)
- new net XIN: C2.2, U2.21 (XIN), Y1.3
- new net XOUT: R5.2, U2.22 (XOUT)
- no-connect marks 0 -> 18
Other:
- note added: "12 MHz Crystal"
- note added: "Buttons"
- note added: "Connectors"
- note added: "Decoupling capacitors for MCU"
- note added: "Flash memory"
- note added: "MicroSD Reader"
- note added: "Microcontroler"
- note added: "PS1 DATA SIGNALS"
- note added: "PS1 POWER SUPPLY"
- note added: "Power MUX"
- note added: "USB POWER SUPPLY"
- note added: "VREG circuit"

Commit message: BOM and Gerber files
Parts:
- removed C20, C21: 100n, Capacitor_SMD:C_0402_1005Metric, symbol Device:C
- removed C23: 1u, Capacitor_SMD:C_0402_1005Metric, symbol Device:C
- removed C25: 4.7u, Capacitor_SMD:C_0402_1005Metric, symbol Device:C
- removed J4: 10118194-0001LF, footprints:AMPHENOL_10118194-0001LF, symbol 10118194-0001LF:10118194-0001LF
- removed R6, R7: 27, Resistor_SMD:R_0402_1005Metric, symbol Device:R
- removed R9: 1k, Resistor_SMD:R_0402_1005Metric, symbol Device:R
- removed U3: TPS2113APWR, footprints:TPS2113-SOP65P640X120-8N, symbol TPS2113APWR:TPS2113APWR
- removed U4: TLV75533PDBVR, footprints:TLV75533PDBVR-SOT95P280X145-5N, symbol TLV75533PDBVR:TLV75533PDBVR
- added TP10: PS1_CMD_DBG, TestPoint:TestPoint_Pad_D1.0mm, symbol Connector:TestPoint
- added TP11: PS1_CS_DBG, TestPoint:TestPoint_Pad_D1.0mm, symbol Connector:TestPoint
- added TP12: PS1_SCK_DBG, TestPoint:TestPoint_Pad_D1.0mm, symbol Connector:TestPoint
- added TP13: PS1_ACK_DBG, TestPoint:TestPoint_Pad_D1.0mm, symbol Connector:TestPoint
- added TP9: PS1_DATA_DBG, TestPoint:TestPoint_Pad_D1.0mm, symbol Connector:TestPoint
- C1, C4: footprint Capacitor_SMD:C_0402_1005Metric -> footprints:C_0402_1005Metric_small_pads
- TP1: Signal (none) -> PS1_DATA
Connections:
- net PS1_3V3 is gone; now on net +3V3: C26.1, U5.5 (OUT)
- net PS1_ACK_DBG: now also TP13.1
- net PS1_CMD_DBG: now also TP10.1
- net PS1_CS_DBG: now also TP11.1
- net PS1_DATA_DBG: now also TP9.1
- net PS1_SCK_DBG: now also TP12.1
- net PS1_3V5: now reaches C27.1, TP8.1, U5.1 (IN), U5.3 (EN)
Other:
- note removed: "Power MUX"
- note removed: "USB POWER SUPPLY"
- moved on the sheet: C26, C27, R13, R14, R15, R16, TP1, TP2, TP3, TP4, TP5, TP6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
