File: hardware/PS-microCard PCB.kicad_sch (KiCad schematic)
At the start: 64 parts, among them J1 Oled Socket, J3 MEM2052-00-195-00-A_REVA, J6 JST Debug Connector, SW1 FSM4JSMA, SW2 FSM4JSMA, U1 W25Q128JVS, U2 RP2350_60QFN, U5 TPS7A2033PDBVR, Y1 ABM8-272-T3

Commit message: new pcb revision
Parts:
- added C20, C21: 1u, Capacitor_SMD:C_0402_1005Metric, symbol Device:C
- added C23, C25, C28: 100n, Capacitor_SMD:C_0402_1005Metric, symbol Device:C
- added J2: 10118194-0001LF, footprints:AMPHENOL_10118194-0001LF, symbol 10118194-0001LF:10118194-0001LF
- added R20: 10k, Resistor_SMD:R_0402_1005Metric, symbol Device:R
- added R21: 20k, Resistor_SMD:R_0402_1005Metric, symbol Device:R
- added R6, R7: 27, Resistor_SMD:R_0402_1005Metric, symbol Device:R
- added R9: 700, Resistor_SMD:R_0402_1005Metric, symbol Device:R
- added U3: TLV75533PDBVR, footprints:TLV75533PDBVR-SOT95P280X145-5N, symbol TLV75533PDBVR:TLV75533PDBVR
- added U4: TPS2113APWR, footprints:TPS2113-SOP65P640X120-8N, symbol TPS2113APWR:TPS2113APWR
Connections:
- net +3V3: now also C28.1, U4.7 (OUT); no longer C26.1, U5.5 (OUT)
- net GND: now also SW2.3, C20.2, C21.1, C23.1, C25.2, C28.2, J2.5 (GND), J2.SH1 (SHIELD), J2.SH2 (SHIELD), J2.SH3 (SHIELD), J2.SH4 (SHIELD), J2.SH5 (SHIELD), J2.SH6 (SHIELD), R20.1, R9.1, U3.2 (GND), U4.2 (~{EN}), U4.5 (GND); no longer S2.2, SW1.2, SW2.1, SW2.2
- net Left Button: now also U2.43 (GPIO29_ADC3); no longer U2.12 (GPIO8)
- net RUN: no longer S1.1
- net Right Button: now also U2.31 (GPIO19); no longer U2.13 (GPIO9)
- net USB_BOOT: no longer S2.3
- net at R17.1, SW1.3: no longer SW1.4
- net at R11.2, S1.3: no longer S1.4
- net D-: now reaches U2.51 (USB_DM)
- net D-: now also R7.2
- net D+: now reaches U2.52 (USB_DP)
- net D+: now also R6.2
- new net: C20.1, J2.1 (VCC), U3.1 (IN), U3.3 (EN)
- new net: R20.2, R21.2, U4.3 (VSNS)
- new net: J2.2 (D-), R7.1
- new net: R9.2, U4.4 (ILIM)
- new net: J2.3 (D+), R6.1
- new net: R18.1, SW2.1
- new net PS1_3V3: C23.2, C26.1, R21.1, U4.8 (IN1), U5.5 (OUT)
- new net USB_3V3: C21.2, C25.1, U3.5 (OUT), U4.6 (IN2)
- now unconnected: SW2.4
- no-connect marks 18 -> 26
Other:
- note added: "Micro USB port"
- note added: "PS1 data signals"
- note added: "PS1 power supply"
- note added: "Power multiplexer"
- note removed: "PS1 DATA SIGNALS"
- note removed: "PS1 POWER SUPPLY"
- moved on the sheet: C1, C2, C3, C4, C5, C6, L1, R1, R18, R2, R3, R4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

Commit message: Revision 1.0A finished
Parts:
- removed J1: Oled Socket, Connector_PinSocket_2.54mm:PinSocket_1x06_P2.54mm_Vertical, symbol Connector_Generic:Conn_01x06
- removed U5: TPS7A2033PDBVR, footprints:TPS7A2033PDBVR-SOT95P280X145-5N, symbol TPS7A2033PDBVR:TPS7A2033PDBVR
- added C29, C30: 220n, Capacitor_SMD:C_0402_1005Metric, symbol Device:C
- added C31, C32, C33, C34: 4.7u, Capacitor_SMD:C_0402_1005Metric, symbol Device:C
- added C35, C36: 10u, Capacitor_SMD:C_0402_1005Metric, symbol Device:C
- added J1: FH12-30S-0.5SH_55_, footprints:HIROSE_FH12-30S-0.5SH_55_, symbol FH12-30S-0.5SH_55_:FH12-30S-0.5SH_55_
- added L2: 4.7u, Inductor_SMD:L_Bourns-SRN4018, symbol Device:L
- added R22: 267k, Resistor_SMD:R_0402_1005Metric, symbol Device:R
- added R23, R24: 10k, Resistor_SMD:R_0402_1005Metric, symbol Device:R
- added R25: 214k, Resistor_SMD:R_0402_1005Metric, symbol Device:R
- added R26, R27: 100k, Resistor_SMD:R_0402_1005Metric, symbol Device:R
- added R28: 20k, Resistor_SMD:R_0402_1005Metric, symbol Device:R
- added TP14: SD_SCK, TestPoint:TestPoint_Pad_D1.0mm, symbol Connector:TestPoint
- added TP15: SD_MISO, TestPoint:TestPoint_Pad_D1.0mm, symbol Connector:TestPoint
- added TP16: SD_CS, TestPoint:TestPoint_Pad_D1.0mm, symbol Connector:TestPoint
- added TP17: SD_DETECT, TestPoint:TestPoint_Pad_D1.0mm, symbol Connector:TestPoint
- added TP18: SD_MOSI, TestPoint:TestPoint_Pad_D1.0mm, symbol Connector:TestPoint
- added U6: MCP1640BT-I_CHY, footprints:SOT95P280X145-6N, symbol MCP1640BT-I_CHY:MCP1640BT-I_CHY
- added U7: TLV75801PDBVR, footprints:SOT95P280X145-5N, symbol TLV75801PDBVR:TLV75801PDBVR
- C27: value 1u -> 10u
- J2: MF FCI Connectors -> Amphenol FCI
- J3: MF Global Connector Technology -> GCT
- J6: MF (none) -> JST Commercial; MP (none) -> SM03B-SRSS-TB (LF)(SN)
- L1: MF (none) -> ABRACON; MP (none) -> AOTA-B201610S3R3-101-T
- R1, R3: now not fitted; now left out of the parts list
- R11: value 1K -> 1k
- R21: value 20k -> 28.7k
- S1, S2: MF TE Connectivity -> TE Connectivity / P&B
- SW1, SW2: MF TE Connectivity -> TE Connectivity / Alcoswitch; MP FSM-4J-SMA -> FSM4JSMA
- TP1, TP10, TP11, TP12, TP13, TP2, TP3, TP4, TP5, TP6, TP7, TP8, TP9: now left out of the parts list
- U1: MF (none) -> Winbond; MP (none) -> W25Q128JVSIQ TR
- U2: MF (none) -> Raspberry Pi; MP (none) -> SC1509(13)-A4
Connections:
- net +3V3: now also C33.2, C35.2, J1.9 (VDD1), L2.1, R23.2, R24.1, U6.3 (EN), U6.6 (VIN)
- net GND: now also C31.1, C32.2, C33.1, C34.1, C35.1, C36.1, J1.10 (IM0), J1.11 (IM1), J1.12 (IM2), J1.8 (VSS), J1.S1 (SHIELD), J1.S2 (SHIELD), R22.2, R26.1, R28.1, U6.2 (GND), U7.2 (GND)
- net OLED_CS: now also J1.13 (CSB), R23.1
- net OLED_D/C: now also J1.15 (A0)
- net OLED_MOSI: now also J1.19 (D1)
- net OLED_SCK: now also J1.18 (D0)
- net PS1_3V3: now also R27.1, U7.5 (OUT)
- net PS1_3V5: now also U7.1 (IN), U7.3 (EN)
- net SD_CS: now also TP16.1
- net SD_DETECT: now also TP17.1
- net SD_MISO: now also TP15.1
- net SD_MOSI: now also TP18.1
- net SD_SCK: now also TP14.1
- net DIFF-: now reaches J2.2 (D-), R7.1
- net OLED_RES: now reaches U2.13 (GPIO9)
- net OLED_RES: now also J1.14 (RESB), R24.2
- net DIFF+: now reaches J2.3 (D+), R6.1
- new net: C29.2, J1.2 (C1N)
- new net: J1.26 (IREF), R22.1
- new net: C32.1, J1.27 (VCOMH)
- new net: C34.2, J1.28 (VPP)
- new net: C29.1, J1.3 (C1P)
- new net: C30.2, J1.4 (C2P)
- new net: C30.1, J1.5 (C2N)
- new net: R27.2, R28.2, U7.4 (FB)
- new net: L2.2, U6.1 (SW)
- new net: R25.2, R26.2, U6.4 (VFB)
- new net OLED_3V8: C31.2, C36.2, J1.6 (VDD2), R25.1, U6.5 (VOUT)
- no-connect marks 26 -> 37
Other:
- note added: "JST connector"
- note added: "Oled connector + Step up converter"
- note removed: "Connectors"
- moved on the sheet: J6, R10, R8

Commit message: BOM update
Parts:
- C1, C13, C26, C31, C32, C33, C34, C4, C6: MF (none) -> KYOCERA AVX; MP (none) -> KGM05CR51A475KH
- C10, C11, C12, C14, C15, C16, C17, C18, C22, C23, C25, C28, C5, C7, C8, C9: MF (none) -> Murata Electronics; MP (none) -> GRM155R71C104KA88D
- C19: MF (none) -> Murata Electronics; MP (none) -> GRM21BR61C106ME15L
- C2, C3: MF (none) -> Murata Electronics; MP (none) -> GRM1555C1H150JA01D
- C20, C21: MF (none) -> Murata Electronics; MP (none) -> GXT155R61A105KE01D
- C24: MF (none) -> TDK; MP (none) -> CGA4J3X7R1A475K125AB
- C27, C29, C30, C35, C36: MF (none) -> Murata Electronics; MP (none) -> GRM155R71C224KA12D
- R10, R20, R23, R24, R8: MF (none) -> YAGEO; MP (none) -> RC0402FR-0710KL
- R11, R17, R18, R19, R5: MF (none) -> YAGEO; MP (none) -> RC0402FR-071KL
- R12, R13, R14, R15, R16: MF (none) -> YAGEO; MP (none) -> RC0402FR-0747RL
- R2: MF (none) -> YAGEO; MP (none) -> RC0402FR-070RL
- R21: MF (none) -> Walsin; MP (none) -> WR04X2872FTL
- R22: MF (none) -> YAGEO; MP (none) -> RC0402FR-07267KL
- R25: MF (none) -> YAGEO; MP (none) -> AA0402FR-07215KL
- R26, R27: MF (none) -> YAGEO; MP (none) -> RC0402FR-07100KL
- R28: MF (none) -> YAGEO; MP (none) -> RC0402FR-0720KL
- R4: MF (none) -> YAGEO; MP (none) -> RC0402FR-0733RL
- R6, R7: MF (none) -> YAGEO; MP (none) -> RC0402FR-0727RL
- R9: MF (none) -> YAGEO; MP (none) -> RC0402FR-07698RL

Commit message: BOM update
Parts:
- C27, C35, C36: MP GRM155R71C224KA12D -> GRM155R60J106ME15D
Changed lines of the file:
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@@
 			)
 		)
-		(property "Datasheet" "https://pim.murata.com/asset/pim4/ceramicCapacitorSMD/GRM155R71C224KA12-01A-EN_PDF_CERAMICCAPACITORSMD"
+		(property "Datasheet" "https://pim.murata.com/asset/pim4/ceramicCapacitorSMD/GRM155R60J106ME15-01A-EN_PDF_CERAMICCAPACITORSMD"
 			(at 204.47 323.85 0)
 			(hide yes)
@@
 			)
 		)
-		(property "MP" "GRM155R71C224KA12D "
+		(property "MP" "GRM155R60J106ME15D"
 			(at 204.47 323.85 0)
 			(hide yes)
@@
 			)
 		)
-		(property "Datasheet" "https://pim.murata.com/asset/pim4/ceramicCapacitorSMD/GRM155R71C224KA12-01A-EN_PDF_CERAMICCAPACITORSMD"
+		(property "Datasheet" "https://pim.murata.com/asset/pim4/ceramicCapacitorSMD/GRM155R60J106ME15-01A-EN_PDF_CERAMICCAPACITORSMD"
 			(at 143.51 321.31 0)
 			(hide yes)
@@
 			)
 		)
-		(property "MP" "GRM155R71C224KA12D "
+		(property "MP" "GRM155R60J106ME15D"
 			(at 143.51 321.31 0)
 			(hide yes)
@@
 			)
 		)
-		(property "Datasheet" "https://pim.murata.com/asset/pim4/ceramicCapacitorSMD/GRM155R71C224KA12-01A-EN_PDF_CERAMICCAPACITORSMD"
+		(property "Datasheet" "https://pim.murata.com/asset/pim4/ceramicCapacitorSMD/GRM155R60J106ME15-01A-EN_PDF_CERAMICCAPACITORSMD"
 			(at 309.88 162.56 0)
 			(hide yes)
@@
 			)
 		)
-		(property "MP" "GRM155R71C224KA12D "
+		(property "MP" "GRM155R60J106ME15D"
 			(at 309.88 162.56 0)
 			(hide yes)

Commit message: Hardware revision 1.1A
Parts:
- removed C19: 10u, Capacitor_SMD:C_0805_2012Metric, symbol Device:C
- removed C26: 4.7u, Capacitor_SMD:C_0402_1005Metric, symbol Device:C
- removed C27: 10u, Capacitor_SMD:C_0402_1005Metric, symbol Device:C
- removed C28: 100n, Capacitor_SMD:C_0402_1005Metric, symbol Device:C
- removed R20: 10k, Resistor_SMD:R_0402_1005Metric, symbol Device:R
- removed R21: 28.7k, Resistor_SMD:R_0402_1005Metric, symbol Device:R
- removed R9: 700, Resistor_SMD:R_0402_1005Metric, symbol Device:R
- removed U3: TLV75533PDBVR, footprints:TLV75533PDBVR-SOT95P280X145-5N, symbol TLV75533PDBVR:TLV75533PDBVR
- removed U4: TPS2113APWR, footprints:TPS2113-SOP65P640X120-8N, symbol TPS2113APWR:TPS2113APWR
- removed U7: TLV75801PDBVR, footprints:SOT95P280X145-5N, symbol TLV75801PDBVR:TLV75801PDBVR
- added C37: 100n, Capacitor_SMD:C_0402_1005Metric_Pad0.74x0.62mm_HandSolder, symbol Device:C
- added C38, C39: 1u, Capacitor_SMD:C_0402_1005Metric_Pad0.74x0.62mm_HandSolder, symbol Device:C
- added L3: 2.2u, footprints:IND_LQH3NPN2R2MMEL, symbol Device:L
- added R29: 100, Resistor_SMD:R_0402_1005Metric_Pad0.72x0.64mm_HandSolder, symbol Device:R
- added R30, R31: 0, Resistor_SMD:R_0402_1005Metric_Pad0.72x0.64mm_HandSolder, symbol Device:R
- added U3: TPS2116DRLR, footprints:TPS2116DRLR, symbol TPS2116DRLR:TPS2116DRLR
- added U5: TPS63001DRCT, footprints:TPS63001DRCT, symbol TPS63001DRCT:TPS63001DRCT
- C1, C4: MF KYOCERA AVX -> TDK; MP KGM05CR51A475KH -> C1005X5R1A475K050BC
- C10, C11, C12, C14, C15, C16, C17, C18, C2, C22, C29, C3, C30, C5, C7, C8, C9: footprint Capacitor_SMD:C_0402_1005Metric -> Capacitor_SMD:C_0402_1005Metric_Pad0.74x0.62mm_HandSolder
- C13, C31, C32, C33, C34, C6: footprint Capacitor_SMD:C_0402_1005Metric -> Capacitor_SMD:C_0402_1005Metric_Pad0.74x0.62mm_HandSolder; MF KYOCERA AVX -> TDK; MP KGM05CR51A475KH -> C1005X5R1A475K050BC
- C20: value 1u -> 10u; footprint Capacitor_SMD:C_0402_1005Metric -> Capacitor_SMD:C_0805_2012Metric_Pad1.18x1.45mm_HandSolder; MF Murata Electronics -> KEMET; MP GXT155R61A105KE01D -> C0805C106M4PACTU
- C21: value 1u -> 100n; footprint Capacitor_SMD:C_0402_1005Metric -> Capacitor_SMD:C_0402_1005Metric_Pad0.74x0.62mm_HandSolder; MP GXT155R61A105KE01D -> GRM155R71C104KA88D
- C23, C25: value 100n -> 10u; footprint Capacitor_SMD:C_0402_1005Metric -> Capacitor_SMD:C_0805_2012Metric_Pad1.18x1.45mm_HandSolder; MF Murata Electronics -> KEMET; MP GRM155R71C104KA88D -> C0805C106M4PACTU
- C24: footprint Capacitor_SMD:C_0805_2012Metric -> Capacitor_SMD:C_0402_1005Metric_Pad0.74x0.62mm_HandSolder; MP CGA4J3X7R1A475K125AB -> C1005X5R1A475K050BC
- C35, C36: footprint Capacitor_SMD:C_0402_1005Metric -> Capacitor_SMD:C_0805_2012Metric_Pad1.18x1.45mm_HandSolder; MF Murata Electronics -> KEMET; MP GRM155R60J106ME15D -> C0805C106M4PACTU
- L2: footprint Inductor_SMD:L_Bourns-SRN4018 -> Inductor_SMD:L_APV_ANR4018; MF Bourns -> TAIYO YUDEN; MP SRN4018BTA-4R7M -> NRS4018T4R7MDGJ
- R10, R11, R12, R13, R14, R15, R16, R17, R18, R19, R2, R23, R24, R26, R4, R5, R6, R7, R8: footprint Resistor_SMD:R_0402_1005Metric -> Resistor_SMD:R_0402_1005Metric_Pad0.72x0.64mm_HandSolder
- R22: footprint Resistor_SMD:R_0402_1005Metric -> Resistor_SMD:R_0402_1005Metric_Pad0.72x0.64mm_HandSolder; MF YAGEO -> PANASONIC; MP RC0402FR-07267KL -> ERJ2RKF2673X
- R25: footprint Resistor_SMD:R_0402_1005Metric -> Resistor_SMD:R_0402_1005Metric_Pad0.72x0.64mm_HandSolder; MF YAGEO -> PANASONIC; MP AA0402FR-07215KL -> ERJ2RKF2153X
- R27: value 100k -> 28.7k; footprint Resistor_SMD:R_0402_1005Metric -> Resistor_SMD:R_0402_1005Metric_Pad0.72x0.64mm_HandSolder; MP RC0402FR-07100KL -> RC0603FR-0728K7L
- R28: value 20k -> 10k; footprint Resistor_SMD:R_0402_1005Metric -> Resistor_SMD:R_0402_1005Metric_Pad0.72x0.64mm_HandSolder; MP RC0402FR-0720KL -> RC0402FR-0710KL
- U1: value W25Q128JVS -> S25FL128LAGMFI010; MF Winbond -> INFINEON TECHNOLOGIES; MP W25Q128JVSIQ TR -> S25FL128LAGMFI010
Connections:
- net +3V3: now also C23.1, C25.1, U5.1 (VOUT), U5.10 (FB)
- net GND: now also C21.2, C23.2, R28.2, C37.2, C38.1, C39.1, R31.1, U3.1 (GND), U5.11 (POWER_PAD), U5.3 (PGND), U5.9 (GND); no longer C21.1, C23.1, R28.1
- net PS1_3V5: now also C38.2, U3.6 (VIN2)
- net USB_5V: now reaches J2.1 (VCC)
- net USB_5V: now also R27.1, C39.2, U3.3 (VIN1), U3.5 (MODE); no longer C20.1
- net at R27.2: now also R28.1, U3.4 (PR1); no longer R28.2
- removed net PS1_3V3: C23.2, R27.1
- removed net USB_3V3: C21.2, C25.1
- new net: L3.1, U5.2 (L2)
- new net: L3.2, U5.4 (L1)
- new net: C21.1, R29.2, R30.2, U5.6 (EN), U5.8 (VINA)
- new net: R30.1, R31.2, U5.7 (PS/SYNC)
- new net V_SYS: C20.1, C37.1, R29.1, U3.2 (VOUT), U3.7 (VOUT), U5.5 (VIN)
Other:
- note added: "Power section"
- note removed: "Power multiplexer"
- moved on the sheet: J2, R6, R7, TP6, TP7, TP8

Commit message: Fix for pcbway and little cleanup
Parts:
- C38, C39: MF Murata Electronics -> SAMSUNG; MP GRM155R71C104KA88D -> CL05A105KO5NNNC
- R1, R3: value DNF -> 0
- R25: value 214k -> 215k
- R27: MP RC0603FR-0728K7L -> RT0402FRE0728K7L
- R31: now left out of the parts list
Changed lines of the file:
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@@
 			)
 		)
-		(property "MP" "RC0603FR-0728K7L"
+		(property "MP" "RT0402FRE0728K7L "
 			(at 317.5 215.9 0)
 			(hide yes)
@@
 			)
 		)
-		(property "MF" "Murata Electronics "
+		(property "MF" "SAMSUNG"
 			(at 317.5 200.66 0)
 			(hide yes)
@@
 			)
 		)
-		(property "MP" "GRM155R71C104KA88D"
+		(property "MP" "CL05A105KO5NNNC "
 			(at 317.5 200.66 0)
 			(hide yes)
@@
 			)
 		)
-		(property "Value" "214k"
+		(property "Value" "215k"
 			(at 175.26 297.18 90)
 			(show_name no)
@@
 		(body_style 1)
 		(exclude_from_sim no)
-		(in_bom yes)
+		(in_bom no)
 		(on_board yes)
 		(in_pos_files yes)
@@
 			)
 		)
-		(property "MF" "Murata Electronics "
+		(property "MF" "SAMSUNG"
 			(at 328.93 200.66 0)
 			(hide yes)
@@
 			)
 		)
-		(property "MP" "GRM155R71C104KA88D"
+		(property "MP" "CL05A105KO5NNNC "
 			(at 328.93 200.66 0)
 			(hide yes)
@@
 			)
 		)
-		(property "Value" "DNF"
+		(property "Value" "0"
 			(at 37.084 116.586 90)
 			(show_name no)
@@
 			)
 		)
-		(property "Value" "DNF"
+		(property "Value" "0"
 			(at 60.96 119.3799 0)
 			(show_name no)
